File: tc_pcb/tc_pcb.kicad_pcb (KiCad board)
At the start: 2 copper layers, 40 x 21 mm, 5 parts, among them J1 Conn_01x05, U1 DS18B20

Commit message: tc_pcb: move to new kicad
Other:
- net class Default removed
- net class TC removed
Changed lines of the file:
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@@
-(kicad_pcb (version 20190516) (host pcbnew "(5.1.0-1195-g1548dcfe8)")
+(kicad_pcb (version 20200628) (host pcbnew "(5.99.0-2364-g42a2f1346)")
   (general
     (thickness 1.6)
@@
     (nets 6)
   )
-  (page "A4")
+  (paper "A4")
   (layers
     (0 "F.Cu" signal)
@@
   )
   (setup
-    (last_trace_width 0.35)
-    (trace_clearance 0.3)
-    (zone_clearance 0.3)
-    (zone_45_only no)
-    (trace_min 0.2)
-    (via_size 0.8)
-    (via_drill 0.4)
-    (via_min_size 0.4)
-    (via_min_drill 0.3)
-    (uvia_size 0.3)
-    (uvia_drill 0.1)
-    (uvias_allowed no)
-    (uvia_min_size 0.2)
-    (uvia_min_drill 0.1)
-    (max_error 0.005)
-    (edge_width 0.05)
-    (segment_width 0.2)
-    (pcb_text_width 0.3)
-    (pcb_text_size 1.5 1.5)
-    (mod_edge_width 0.12)
-    (mod_text_size 1 1)
-    (mod_text_width 0.15)
-    (pad_size 1.3 1.3)
-    (pad_drill 0.75)
-    (pad_to_mask_clearance 0.051)
-    (solder_mask_min_width 0.25)
-    (aux_axis_origin 0 0)
     (grid_origin 140.63 105.37)
-    (visible_elements FFFFFF7F)
     (pcbplotparams
       (layerselection 0x010fc_ffffffff)
@@
       (usegerberadvancedattributes false)
       (creategerberjobfile false)
+      (svguseinch false)
+      (svgprecision 6)
       (excludeedgelayer true)
       (linewidth 0.100000)
@@
       (plotvalue true)
       (plotinvisibletext false)
-      (padsonsilk false)
+      (sketchpadsonfab false)
       (subtractmaskfromsilk false)
       (outputformat 1)
@@
       (drillshape 0)
       (scaleselection 1)
-      (outputdirectory ""))
+      (outputdirectory "")
+    )
   )
   (net 0 "")
@@
   (net 4 "GND")
   (net 5 "/TC-")
-  (net_class "Default" "Это класс цепей по умолчанию."
-    (clearance 0.3)
-    (trace_width 0.35)
-    (via_dia 0.8)
-    (via_drill 0.4)
-    (uvia_dia 0.3)
-    (uvia_drill 0.1)
-    (add_net "+5V")
-    (add_net "/DQ")
-    (add_net "/TC+")
-    (add_net "/TC-")
-    (add_net "GND")
-  )
-  (net_class "TC" ""
-    (clearance 0.3)
-    (trace_width 0.75)
-    (via_dia 0.8)
-    (via_drill 0.4)
-    (uvia_dia 0.3)
-    (uvia_drill 0.1)
-  )
   (module "Package_TO_SOT_THT:TO-92_W4.0mm_StaggerEven_Horizontal_FlatSideDown" (layer "B.Cu")
-    (at 141.9 104.1 270)
+    (at 141.9 104.1 -90)
     (descr "TO-92 horizontal, leads molded, narrow, drill 0.75mm (see NXP sot054_po.pdf)")
     (tags "to-92 sc-43 sc-43a sot54 PA33 transistor")
@@
     (fp_line (start 1.27 -3.94) (end 1.27 1.27) (layer "B.Fab") (width 0.1))
     (fp_line (start 2.54 -3.94) (end 2.54 0) (layer "B.Fab") (width 0.1))
-    (fp_text user "%R" (at 1.27 -6.6 90) (layer "B.Fab")
+    (fp_text user "${REFERENCE}" (at 1.27 -6.6 90) (layer "B.Fab")
       (effects (font (size 1 1) (thickness 0.15)) (justify mirror))
     )
@@
   )
   (module "Connector_PinSocket_2.54mm:PinSocket_1x05_P2.54mm_Vertical" locked (layer "F.Cu")
-    (at 157.4 109.6 270)
+    (at 157.4 109.6 -90)
     (descr "Through hole straight socket strip, 1x05, 2.54mm pitch, single row (from Kicad 4.0.7), script generated")
     (tags "Through hole socket strip THT 1x05 2.54mm single row")
@@
     (fp_line (start 1.75 11.9) (end -1.8 11.9) (layer "F.CrtYd") (width 0.05))
     (fp_line (start -1.8 11.9) (end -1.8 -1.8) (layer "F.CrtYd") (width 0.05))
-    (fp_text user "%R" (at 0 5.08) (layer "F.Fab")
-      (effects (font (size 1 1) (thickness 0.15)))
-    )
+    (fp_text user "${REFERENCE}" (at 0 5.08) (layer "F.Fab")
+      (effects (font (size 1 1) (thickness 0.15)))
+    )
